File: EEGAmp_SMT_MountHole.brd (EAGLE design)
At the start: 25.5 x 11.2 mm, 15 parts, among them U1 TL084QD

Commit message: fixed, smaller
Parts:
- moved R5 1.52 mm to (28.7, 29.7)
- moved R6 1.02 mm to (26.3, 29.7)
- moved AIN- 0.64 mm to (19.7, 20.8)
Routing:
- net VDD: track 25.0 -> 12.8 mm, vias 0 -> 1
- net GND: track 27.6 -> 24.3 mm, vias 1 -> 2
- net VOD: track 13.5 -> 14.1 mm
- net VREF: track 12.2 -> 11.6 mm
Other:
- board size 25.5 x 11.2 mm -> 23.2 x 11.3 mm
