File: EEGAmp_SMT_MountHole.brd (EAGLE design)
At the start: 23.2 x 11.3 mm, 15 parts, among them U1 TL084QD

Commit message: another wire tolerance fix
Routing:
- net VOD: track 14.1 -> 13.2 mm
Changed lines of the file:
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@@
 <wire x1="31.2674" y1="24.4122" x2="31.2674" y2="27.7698" width="0.1524" layer="16"/>
 <wire x1="31.2674" y1="27.7698" x2="31.3106" y2="27.813" width="0.1524" layer="16"/>
-<wire x1="31.3106" y1="27.813" x2="31.0086" y2="28.115" width="0.1524" layer="1"/>
-<wire x1="31.0086" y1="28.115" x2="31.0086" y2="28.86681875" width="0.1524" layer="1"/>
-<wire x1="31.0086" y1="28.86681875" x2="30.18815" y2="29.68726875" width="0.1524" layer="1"/>
+<wire x1="31.3106" y1="27.813" x2="31.1356" y2="27.988" width="0.1524" layer="1"/>
+<wire x1="31.1356" y1="27.988" x2="31.1356" y2="28.73981875" width="0.1524" layer="1"/>
+<wire x1="31.1356" y1="28.73981875" x2="30.18815" y2="29.68726875" width="0.1524" layer="1"/>
 <wire x1="30.18815" y1="29.68726875" x2="29.202040625" y2="29.68726875" width="0.1524" layer="1"/>
 <wire x1="29.202040625" y1="29.68726875" x2="29.202" y2="29.718" width="0" layer="19" extent="1-1"/>
@@
 <contactref element="R7" pad="1"/>
 <contactref element="R4" pad="2"/>
-<wire x1="21.4042" y1="24.4094" x2="21.4042" y2="25.9588" width="0.1524" layer="1"/>
+<wire x1="21.4042" y1="24.4094" x2="22.9536" y2="25.9588" width="0.1524" layer="1"/>
 <wire x1="21.4042" y1="25.4508" x2="21.4042" y2="24.4094" width="0.1524" layer="1"/>
-<wire x1="21.4042" y1="25.9588" x2="29.5402" y2="25.9588" width="0.1524" layer="1"/>
+<wire x1="22.9536" y1="25.9588" x2="29.5402" y2="25.9588" width="0.1524" layer="1"/>
 <wire x1="30.48" y1="25.019" x2="30.48" y2="22.925" width="0.1524" layer="1"/>
 <wire x1="29.5402" y1="25.9588" x2="30.48" y2="25.019" width="0.1524" layer="1"/>
