File: EEGAmp_SMT_MountHole.brd (EAGLE design)
At the start: 23.2 x 11.3 mm, 15 parts, among them U1 TL084QD

Commit message: fixed reference circuit (oops)
Parts:
- added REFOUT: PTR1PAD1-17, testpad:P1-17
- moved C2 2.43 mm to (23.6, 29.7), turned to 180 degrees
- moved R8 1.41 mm to (21.6, 29.3)
- moved AIN- 0.23 mm to (19.5, 20.8)
- moved C1 0.23 mm to (20.8, 26.6)
- moved JP2 0.15 mm to (33.2, 25.3)
Connections:
- new net REFOUT: REFOUT.TP, U1.12, U1.8, U1.9
- net GND: no longer R5.2
- net VREF: now also R5.2; no longer U1.12, U1.8, U1.9
Routing:
- net REFOUT: track 0.00 -> 17.2 mm, vias 0 -> 1
- net VREF: track 11.6 -> 5.69 mm
- net GND: track 24.3 -> 27.4 mm, vias 2 -> 1
- net VDD: track 12.9 -> 14.0 mm
