File: EEGAmp_SMT.sch (EAGLE design)
At the start: 14 parts, among them U1 TL084QD

Commit message: fixed reference circuit (oops)
Parts:
- removed JP1: (no value), pinhead:PINHD-1X2
- added JP3: (no value), pinhead:PINHD-1X3
Connections:
- new net REFOUT: JP3.1, U1.3IN-, U1.3OUT, U1.4IN+
- net AIN+: now also JP3.2; no longer JP1.1
- net AIN-: now also JP3.3; no longer JP1.2
- net GND: no longer R5.2
- net VREF: now also R5.2; no longer U1.3IN-, U1.3OUT, U1.4IN+
