File: EEGAmp_SMT_MountHole.sch (EAGLE design)
At the start: 15 parts, among them U1 TL084QD

Commit message: fixed reference circuit (oops)
Parts:
- added REFOUT: PTR1PAD1-17, testpad:PTR1PAD1-17
Connections:
- new net REFOUT: REFOUT.TP, U1.3IN-, U1.3OUT, U1.4IN+
- net GND: no longer R5.2
- net VREF: now also R5.2; no longer U1.3IN-, U1.3OUT, U1.4IN+
