File: EEGAmp_Thruhole.brd (EAGLE design)
At the start: 30 x 21.6 mm, 14 parts, among them U1 TL084BCN

Commit message: fixed reference circuit (oops)
Parts:
- JP1: device pinhead:1X02 -> pinhead:1X03
- moved JP1 0.15 mm to (14.7, 25.3)
Connections:
- new net REFOUT: JP1.1, U1.12, U1.8, U1.9
- net AIN+: now also JP1.2; no longer JP1.1
- net AIN-: now also JP1.3; no longer JP1.2
- net GND: no longer R5.2
- net VREF: now also R5.2; no longer U1.12, U1.8, U1.9
Routing:
- net REFOUT: track 0.00 -> 25.3 mm, vias 0 -> 1
- net VREF: track 20.3 -> 27.6 mm, vias 0 -> 1
- net GND: track 41.6 -> 43.7 mm
- net AIN+: track 16.9 -> 16.1 mm
- net AIN-: track 10.7 -> 9.96 mm
- net VDD: track 28.5 -> 29.1 mm
- net AOUT: track 32.1 -> 31.6 mm
Other:
- board text added: "REFOUT"
