File: EEGAmp_Thruhole.sch (EAGLE design)
At the start: 14 parts, among them U1 TL084BCN

Commit message: fixed reference circuit (oops)
Parts:
- JP1: device pinhead:PINHD-1X2 -> pinhead:PINHD-1X3
Connections:
- new net REFOUT: JP1.1, U1.3IN-, U1.3OUT, U1.4IN+
- net AIN+: now also JP1.2; no longer JP1.1
- net AIN-: now also JP1.3; no longer JP1.2
- net GND: no longer R5.2
- net VREF: now also R5.2; no longer U1.3IN-, U1.3OUT, U1.4IN+
Changed lines of the file:
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@@
 <part name="SUPPLY2" library="supply2" library_urn="urn:adsk.eagle:library:372" deviceset="GND" device=""/>
 <part name="C3" library="capacitor-wima" library_urn="urn:adsk.eagle:library:116" deviceset="C" device="2.5/2" package3d_urn="urn:adsk.eagle:package:5415/1"/>
-<part name="SUPPLY3" library="supply2" library_urn="urn:adsk.eagle:library:372" deviceset="GND" device=""/>
 <part name="SUPPLY4" library="supply2" library_urn="urn:adsk.eagle:library:372" deviceset="GND" device=""/>
-<part name="JP1" library="pinhead" library_urn="urn:adsk.eagle:library:325" deviceset="PINHD-1X2" device="" package3d_urn="urn:adsk.eagle:package:22435/2"/>
 <part name="JP2" library="pinhead" library_urn="urn:adsk.eagle:library:325" deviceset="PINHD-1X4" device="" package3d_urn="urn:adsk.eagle:package:22407/2"/>
+<part name="JP1" library="pinhead" library_urn="urn:adsk.eagle:library:325" deviceset="PINHD-1X3" device="" package3d_urn="urn:adsk.eagle:package:22458/2"/>
 </parts>
 <sheets>
@@
 <attribute name="VALUE" x="197.104" y="84.201" size="1.778" layer="96"/>
 </instance>
-<instance part="SUPPLY3" gate="GND" x="55.88" y="58.42" smashed="yes" rot="R270">
-<attribute name="VALUE" x="53.975" y="52.705" size="1.778" layer="96"/>
-</instance>
 <instance part="SUPPLY4" gate="GND" x="104.14" y="58.42" smashed="yes" rot="R90">
 <attribute name="VALUE" x="102.235" y="52.705" size="1.778" layer="96"/>
-</instance>
-<instance part="JP1" gate="G$1" x="142.24" y="30.48" smashed="yes" rot="R180">
-<attribute name="NAME" x="148.59" y="24.765" size="1.778" layer="95" rot="R180"/>
-<attribute name="VALUE" x="148.59" y="35.56" size="1.778" layer="96" rot="R180"/>
 </instance>
 <instance part="JP2" gate="A" x="236.22" y="73.66" smashed="yes">
 <attribute name="NAME" x="229.87" y="81.915" size="1.778" layer="95"/>
 <attribute name="VALUE" x="229.87" y="66.04" size="1.778" layer="96"/>
+</instance>
+<instance part="JP1" gate="A" x="142.24" y="27.94" smashed="yes" rot="R180">
+<attribute name="NAME" x="148.59" y="22.225" size="1.778" layer="95" rot="R180"/>
+<attribute name="VALUE" x="148.59" y="35.56" size="1.778" layer="96" rot="R180"/>
 </instance>
 </instances>
@@
 </segment>
 <segment>
-<pinref part="R5" gate="G$1" pin="2"/>
-<wire x1="63.5" y1="58.42" x2="58.42" y2="58.42" width="0.1524" layer="91"/>
-<pinref part="SUPPLY3" gate="GND" pin="GND"/>
-</segment>
-<segment>
 <pinref part="R6" gate="G$1" pin="1"/>
 <wire x1="96.52" y1="58.42" x2="101.6" y2="58.42" width="0.1524" layer="91"/>
@@
 </segment>
 <segment>
-<pinref part="JP1" gate="G$1" pin="2"/>
 <wire x1="144.78" y1="30.48" x2="152.4" y2="30.48" width="0.1524" layer="91"/>
 <label x="152.4" y="30.48" size="1.778" layer="95"/>
+<pinref part="JP1" gate="A" pin="3"/>
 </segment>
 </net>
 <net name="VREF" class="0">
-<segment>
-<pinref part="U1" gate="A" pin="4IN+"/>
-<wire x1="152.4" y1="58.42" x2="147.32" y2="58.42" width="0.1524" layer="91"/>
-<label x="139.7" y="58.42" size="1.778" layer="95"/>
-</segment>
-<segment>
-<pinref part="U1" gate="A" pin="3OUT"/>
-<wire x1="187.96" y1="68.58" x2="193.04" y2="68.58" width="0.1524" layer="91"/>
-<label x="193.04" y="68.58" size="1.778" layer="95"/>
-</segment>
-<segment>
-<pinref part="U1" gate="A" pin="3IN-"/>
-<wire x1="152.4" y1="60.96" x2="147.32" y2="60.96" width="0.1524" layer="91"/>
-<label x="139.7" y="60.96" size="1.778" layer="95"/>
-</segment>
 <segment>
 <pinref part="JP2" gate="A" pin="2"/>
@@
 <label x="220.98" y="76.2" size="1.778" layer="95"/>
 </segment>
+<segment>
+<pinref part="R5" gate="G$1" pin="2"/>
+<wire x1="63.5" y1="58.42" x2="58.42" y2="58.42" width="0.1524" layer="91"/>
+<label x="53.34" y="58.42" size="1.778" layer="95"/>
+</segment>
 </net>
 <net name="AIN+" class="0">
@@
 </segment>
 <segment>
-<pinref part="JP1" gate="G$1" pin="1"/>
 <wire x1="144.78" y1="27.94" x2="152.4" y2="27.94" width="0.1524" layer="91"/>
 <label x="152.4" y="27.94" size="1.778" layer="95"/>
+<pinref part="JP1" gate="A" pin="2"/>
 </segment>
 </net>
@@
 </segment>
 </net>
+<net name="REFOUT" class="0">
+<segment>
+<pinref part="JP1" gate="A" pin="1"/>
+<wire x1="144.78" y1="25.4" x2="152.4" y2="25.4" width="0.1524" layer="91"/>
+<label x="152.4" y="25.4" size="1.778" layer="95"/>
+</segment>
+<segment>
+<pinref part="U1" gate="A" pin="3IN-"/>
+<wire x1="152.4" y1="60.96" x2="147.32" y2="60.96" width="0.1524" layer="91"/>
+<label x="139.7" y="60.96" size="1.778" layer="95"/>
+</segment>
+<segment>
+<pinref part="U1" gate="A" pin="4IN+"/>
+<wire x1="152.4" y1="58.42" x2="147.32" y2="58.42" width="0.1524" layer="91"/>
+<label x="139.7" y="58.42" size="1.778" layer="95"/>
+</segment>
+<segment>
+<pinref part="U1" gate="A" pin="3OUT"/>
+<wire x1="187.96" y1="68.58" x2="193.04" y2="68.58" width="0.1524" layer="91"/>
+<label x="193.04" y="68.58" size="1.778" layer="95"/>
+</segment>
+</net>
