File: CAD/singular_amps/Amplifiers.brd (EAGLE design)
At the start: 16 parts, among them U1 TL082CP, U2 TL081CP, U3 TL081CP

Commit message: fix
Connections:
- new net REFOUT: U2.2, U2.6, U3.3
- net GND: no longer R5.2
- net VREF: now also R5.2; no longer U2.2, U2.6, U3.3
Changed lines of the file:
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@@
 <signal name="GND">
 <contactref element="R2" pad="1"/>
-<contactref element="R5" pad="2"/>
 <contactref element="R6" pad="1"/>
 <contactref element="C3" pad="1"/>
 <contactref element="C4" pad="1"/>
 <contactref element="C5" pad="1"/>
-<wire x1="6.35" y1="11.43" x2="6.35" y2="6.35" width="0" layer="19" extent="1-1"/>
-<wire x1="6.35" y1="16.51" x2="6.35" y2="11.43" width="0" layer="19" extent="1-1"/>
-<wire x1="36.83" y1="25.4" x2="6.35" y2="16.51" width="0" layer="19" extent="1-1"/>
-<wire x1="36.83" y1="33.02" x2="36.83" y2="25.4" width="0" layer="19" extent="1-1"/>
-<wire x1="49.53" y1="29.21" x2="36.83" y2="25.4" width="0" layer="19" extent="1-1"/>
+<wire x1="36.83" y1="25.4" x2="36.83" y2="33.02" width="0" layer="19" extent="1-1"/>
+<wire x1="6.35" y1="16.51" x2="36.83" y2="25.4" width="0" layer="19" extent="1-1"/>
+<wire x1="6.35" y1="11.43" x2="6.35" y2="16.51" width="0" layer="19" extent="1-1"/>
+<wire x1="6.35" y1="6.35" x2="6.35" y2="11.43" width="0" layer="19" extent="1-1"/>
 </signal>
 <signal name="N$9">
@@
 </signal>
 <signal name="VREF">
-<contactref element="U2" pad="6"/>
-<contactref element="U2" pad="2"/>
-<contactref element="U3" pad="3"/>
-<wire x1="16.35" y1="29.21" x2="24.29" y2="26.67" width="0" layer="19" extent="1-1"/>
-<wire x1="6.19" y1="26.67" x2="16.35" y2="29.21" width="0" layer="19" extent="1-1"/>
+<contactref element="R5" pad="2"/>
 </signal>
 <signal name="N$7">
@@
 <wire x1="8.89" y1="16.51" x2="8.89" y2="11.43" width="0" layer="19" extent="1-1"/>
 </signal>
+<signal name="REFOUT">
+<contactref element="U3" pad="3"/>
+<contactref element="U2" pad="6"/>
+<contactref element="U2" pad="2"/>
+<wire x1="16.35" y1="29.21" x2="24.29" y2="26.67" width="0" layer="19" extent="1-1"/>
+<wire x1="6.19" y1="26.67" x2="16.35" y2="29.21" width="0" layer="19" extent="1-1"/>
+</signal>
 </signals>

Commit message: corrected notes
Parts:
- added JP2: (no value), pinhead:1X04
- added JP3: (no value), pinhead:1X03
Connections:
- net AIN+: now also JP3.2
- net AIN-: now also JP3.3
- net AOUT: now also JP2.4
- net GND: now also JP2.3
- net REFOUT: now also JP3.1
- net VDD: now also JP2.1
- net VREF: now also JP2.2
Changed lines of the file:
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@@
 <attribute name="VALUE" x="5.969" y="3.556" size="1.27" layer="27" ratio="10"/>
+</element>
+<element name="JP3" library="pinhead" library_urn="urn:adsk.eagle:library:325" package="1X03" package3d_urn="urn:adsk.eagle:package:22458/2" value="" x="10.16" y="1.27" smashed="yes">
+<attribute name="NAME" x="6.2738" y="3.0988" size="1.27" layer="25" ratio="10"/>
+<attribute name="POPULARITY" value="92" x="10.16" y="1.27" size="1.778" layer="27" display="off"/>
+<attribute name="VALUE" x="6.35" y="-1.905" size="1.27" layer="27"/>
+</element>
+<element name="JP2" library="pinhead" library_urn="urn:adsk.eagle:library:325" package="1X04" package3d_urn="urn:adsk.eagle:package:22407/2" value="" x="11.43" y="-5.08" smashed="yes">
+<attribute name="NAME" x="6.2738" y="-3.2512" size="1.27" layer="25" ratio="10"/>
+<attribute name="POPULARITY" value="91" x="11.43" y="-5.08" size="1.778" layer="27" display="off"/>
+<attribute name="VALUE" x="6.35" y="-8.255" size="1.27" layer="27"/>
 </element>
 </elements>
@@
 <contactref element="C4" pad="1"/>
 <contactref element="C5" pad="1"/>
+<contactref element="JP2" pad="3"/>
 <wire x1="36.83" y1="25.4" x2="36.83" y2="33.02" width="0" layer="19" extent="1-1"/>
 <wire x1="6.35" y1="16.51" x2="36.83" y2="25.4" width="0" layer="19" extent="1-1"/>
 <wire x1="6.35" y1="11.43" x2="6.35" y2="16.51" width="0" layer="19" extent="1-1"/>
 <wire x1="6.35" y1="6.35" x2="6.35" y2="11.43" width="0" layer="19" extent="1-1"/>
+<wire x1="12.7" y1="-5.08" x2="6.35" y2="6.35" width="0" layer="19" extent="1-1"/>
 </signal>
 <signal name="N$9">
@@
 <contactref element="R8" pad="2"/>
 <contactref element="U3" pad="6"/>
-<wire x1="41.91" y1="21.59" x2="14.13" y2="26.67" width="0" layer="19" extent="1-1"/>
-<wire x1="44.45" y1="38.1" x2="41.91" y2="21.59" width="0" layer="19" extent="1-1"/>
+<contactref element="JP2" pad="4"/>
+<wire x1="41.91" y1="21.59" x2="44.45" y2="38.1" width="0" layer="19" extent="1-1"/>
+<wire x1="14.13" y1="26.67" x2="41.91" y2="21.59" width="0" layer="19" extent="1-1"/>
+<wire x1="15.24" y1="-5.08" x2="14.13" y2="26.67" width="0" layer="19" extent="1-1"/>
 </signal>
 <signal name="VOD">
@@
 <signal name="VREF">
 <contactref element="R5" pad="2"/>
+<contactref element="JP2" pad="2"/>
+<wire x1="10.16" y1="-5.08" x2="49.53" y2="29.21" width="0" layer="19" extent="1-1"/>
 </signal>
 <signal name="N$7">
@@
 <signal name="AIN-">
 <contactref element="U1" pad="3"/>
+<contactref element="JP3" pad="3"/>
+<wire x1="12.7" y1="1.27" x2="26.51" y2="26.67" width="0" layer="19" extent="1-1"/>
 </signal>
 <signal name="AIN+">
 <contactref element="U1" pad="2"/>
+<contactref element="JP3" pad="2"/>
+<wire x1="10.16" y1="1.27" x2="26.51" y2="29.21" width="0" layer="19" extent="1-1"/>
 </signal>
 <signal name="VDD">
@@
 <contactref element="C4" pad="2"/>
 <contactref element="C5" pad="2"/>
-<wire x1="8.89" y1="11.43" x2="8.89" y2="6.35" width="0" layer="19" extent="1-1"/>
-<wire x1="8.89" y1="16.51" x2="8.89" y2="11.43" width="0" layer="19" extent="1-1"/>
+<contactref element="JP2" pad="1"/>
+<wire x1="8.89" y1="11.43" x2="8.89" y2="16.51" width="0" layer="19" extent="1-1"/>
+<wire x1="8.89" y1="6.35" x2="8.89" y2="11.43" width="0" layer="19" extent="1-1"/>
+<wire x1="7.62" y1="-5.08" x2="8.89" y2="6.35" width="0" layer="19" extent="1-1"/>
 </signal>
 <signal name="REFOUT">
@@
 <contactref element="U2" pad="6"/>
 <contactref element="U2" pad="2"/>
+<contactref element="JP3" pad="1"/>
 <wire x1="16.35" y1="29.21" x2="24.29" y2="26.67" width="0" layer="19" extent="1-1"/>
 <wire x1="6.19" y1="26.67" x2="16.35" y2="29.21" width="0" layer="19" extent="1-1"/>
+<wire x1="7.62" y1="1.27" x2="6.19" y2="26.67" width="0" layer="19" extent="1-1"/>
 </signal>
 </signals>
