File: CAD/singular_amps/Amplifiers.sch (EAGLE design)
At the start: 16 parts, among them U1 TL082CP, U2 TL081CP, U3 TL081CP

Commit message: fix
Connections:
- new net REFOUT: U2.IN-, U2.OUT, U3.IN_+
- net GND: no longer R5.2
- net VREF: now also R5.2; no longer U2.IN-, U2.OUT, U3.IN_+
Changed lines of the file:
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@@
 <part name="C2" library="capacitor-wima" library_urn="urn:adsk.eagle:library:116" deviceset="C" device="2.5/2" package3d_urn="urn:adsk.eagle:package:5415/1"/>
 <part name="SUPPLY1" library="supply2" library_urn="urn:adsk.eagle:library:372" deviceset="GND" device=""/>
-<part name="SUPPLY3" library="supply2" library_urn="urn:adsk.eagle:library:372" deviceset="GND" device=""/>
 <part name="SUPPLY4" library="supply2" library_urn="urn:adsk.eagle:library:372" deviceset="GND" device=""/>
 <part name="U1" library="TL082CP" deviceset="TL082CP" device=""/>
@@
 <attribute name="VALUE" x="40.005" y="79.375" size="1.778" layer="96"/>
 </instance>
-<instance part="SUPPLY3" gate="GND" x="62.23" y="54.61" smashed="yes" rot="R270">
-<attribute name="VALUE" x="60.325" y="48.895" size="1.778" layer="96"/>
-</instance>
 <instance part="SUPPLY4" gate="GND" x="110.49" y="54.61" smashed="yes" rot="R90">
 <attribute name="VALUE" x="108.585" y="48.895" size="1.778" layer="96"/>
@@
 <wire x1="41.91" y1="90.17" x2="41.91" y2="85.09" width="0.1524" layer="91"/>
 <pinref part="SUPPLY1" gate="GND" pin="GND"/>
-</segment>
-<segment>
-<pinref part="R5" gate="G$1" pin="2"/>
-<wire x1="69.85" y1="54.61" x2="64.77" y2="54.61" width="0.1524" layer="91"/>
-<pinref part="SUPPLY3" gate="GND" pin="GND"/>
 </segment>
 <segment>
@@
 <net name="VREF" class="0">
 <segment>
-<pinref part="U2" gate="A" pin="OUT"/>
-<wire x1="190.5" y1="60.96" x2="194.31" y2="60.96" width="0.1524" layer="91"/>
-<label x="195.58" y="59.69" size="1.778" layer="95"/>
-</segment>
-<segment>
-<pinref part="U2" gate="A" pin="IN-"/>
-<wire x1="154.94" y1="60.96" x2="152.4" y2="60.96" width="0.1524" layer="91"/>
-<label x="146.05" y="60.96" size="1.778" layer="95"/>
-</segment>
-<segment>
-<pinref part="U3" gate="A" pin="IN_+"/>
-<wire x1="154.94" y1="24.13" x2="151.13" y2="24.13" width="0.1524" layer="91"/>
-<label x="143.51" y="22.86" size="1.778" layer="95"/>
+<pinref part="R5" gate="G$1" pin="2"/>
+<wire x1="69.85" y1="54.61" x2="64.77" y2="54.61" width="0.1524" layer="91"/>
+<label x="60.96" y="55.88" size="1.778" layer="95"/>
 </segment>
 </net>
@@
 </segment>
 </net>
+<net name="REFOUT" class="0">
+<segment>
+<pinref part="U3" gate="A" pin="IN_+"/>
+<wire x1="154.94" y1="24.13" x2="151.13" y2="24.13" width="0.1524" layer="91"/>
+<label x="143.51" y="22.86" size="1.778" layer="95"/>
+</segment>
+<segment>
+<pinref part="U2" gate="A" pin="OUT"/>
+<wire x1="190.5" y1="60.96" x2="194.31" y2="60.96" width="0.1524" layer="91"/>
+<label x="195.58" y="59.69" size="1.778" layer="95"/>
+</segment>
+<segment>
+<pinref part="U2" gate="A" pin="IN-"/>
+<wire x1="154.94" y1="60.96" x2="152.4" y2="60.96" width="0.1524" layer="91"/>
+<label x="146.05" y="60.96" size="1.778" layer="95"/>
+</segment>
+</net>

Commit message: corrected notes
Parts:
- added JP2: (no value), pinhead:PINHD-1X4
- added JP3: (no value), pinhead:PINHD-1X3
Connections:
- net AIN+: now also JP3.2
- net AIN-: now also JP3.3
- net AOUT: now also JP2.4
- net GND: now also JP2.3
- net REFOUT: now also JP3.1
- net VDD: now also JP2.1
- net VREF: now also JP2.2
Other:
- note added: "VRef can be VDD or a dedicated voltage reference for the ADC"
Changed lines of the file:
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@@
 <part name="SUPPLY5" library="supply2" library_urn="urn:adsk.eagle:library:372" deviceset="GND" device=""/>
 <part name="SUPPLY6" library="supply2" library_urn="urn:adsk.eagle:library:372" deviceset="GND" device=""/>
+<part name="JP3" library="pinhead" library_urn="urn:adsk.eagle:library:325" deviceset="PINHD-1X3" device="" package3d_urn="urn:adsk.eagle:package:22458/2"/>
+<part name="JP2" library="pinhead" library_urn="urn:adsk.eagle:library:325" deviceset="PINHD-1X4" device="" package3d_urn="urn:adsk.eagle:package:22407/2"/>
 </parts>
 <sheets>
@@
 R7: 1kΩ
 R8: 1MΩ</text>
+<text x="205.74" y="-5.08" size="1.778" layer="97">VRef can be VDD or a dedicated voltage reference for the ADC</text>
 </plain>
 <instances>
@@
 <attribute name="VALUE" x="215.265" y="81.915" size="1.778" layer="96"/>
 </instance>
+<instance part="JP3" gate="A" x="132.08" y="-15.24" smashed="yes" rot="R180">
+<attribute name="NAME" x="138.43" y="-20.955" size="1.778" layer="95" rot="R180"/>
+<attribute name="VALUE" x="138.43" y="-7.62" size="1.778" layer="96" rot="R180"/>
+</instance>
+<instance part="JP2" gate="A" x="223.52" y="-17.78" smashed="yes">
+<attribute name="NAME" x="217.17" y="-9.525" size="1.778" layer="95"/>
+<attribute name="VALUE" x="217.17" y="-25.4" size="1.778" layer="96"/>
+</instance>
 </instances>
 <busses>
@@
 <wire x1="194.31" y1="87.63" x2="217.17" y2="87.63" width="0.1524" layer="91"/>
 <pinref part="SUPPLY6" gate="GND" pin="GND"/>
+</segment>
+<segment>
+<pinref part="JP2" gate="A" pin="3"/>
+<wire x1="220.98" y1="-17.78" x2="213.36" y2="-17.78" width="0.1524" layer="91"/>
+<label x="208.28" y="-17.78" size="1.778" layer="95"/>
 </segment>
 </net>
@@
 <wire x1="190.5" y1="26.67" x2="194.31" y2="26.67" width="0.1524" layer="91"/>
 <label x="194.31" y="26.67" size="1.778" layer="95"/>
+</segment>
+<segment>
+<pinref part="JP2" gate="A" pin="4"/>
+<wire x1="220.98" y1="-20.32" x2="213.36" y2="-20.32" width="0.1524" layer="91"/>
+<label x="208.28" y="-20.32" size="1.778" layer="95"/>
 </segment>
 </net>
@@
 <label x="60.96" y="55.88" size="1.778" layer="95"/>
 </segment>
+<segment>
+<pinref part="JP2" gate="A" pin="2"/>
+<wire x1="220.98" y1="-15.24" x2="213.36" y2="-15.24" width="0.1524" layer="91"/>
+<label x="208.28" y="-15.24" size="1.778" layer="95"/>
+</segment>
 </net>
 <net name="N$7" class="0">
@@
 <label x="147.32" y="102.87" size="1.778" layer="95"/>
 </segment>
+<segment>
+<wire x1="134.62" y1="-12.7" x2="142.24" y2="-12.7" width="0.1524" layer="91"/>
+<label x="142.24" y="-12.7" size="1.778" layer="95"/>
+<pinref part="JP3" gate="A" pin="3"/>
+</segment>
 </net>
 <net name="AIN+" class="0">
@@
 <wire x1="154.94" y1="97.79" x2="152.4" y2="97.79" width="0.1524" layer="91"/>
 <label x="147.32" y="97.79" size="1.778" layer="95"/>
+</segment>
+<segment>
+<wire x1="134.62" y1="-15.24" x2="142.24" y2="-15.24" width="0.1524" layer="91"/>
+<label x="142.24" y="-15.24" size="1.778" layer="95"/>
+<pinref part="JP3" gate="A" pin="2"/>
 </segment>
 </net>
@@
 <label x="207.01" y="34.29" size="1.778" layer="95"/>
 </segment>
+<segment>
+<pinref part="JP2" gate="A" pin="1"/>
+<wire x1="220.98" y1="-12.7" x2="213.36" y2="-12.7" width="0.1524" layer="91"/>
+<label x="208.28" y="-12.7" size="1.778" layer="95"/>
+</segment>
 </net>
 <net name="REFOUT" class="0">
@@
 <label x="146.05" y="60.96" size="1.778" layer="95"/>
 </segment>
-</net>
+<segment>
+<pinref part="JP3" gate="A" pin="1"/>
+<wire x1="134.62" y1="-17.78" x2="142.24" y2="-17.78" width="0.1524" layer="91"/>
+<label x="142.24" y="-17.78" size="1.778" layer="95"/>
+</segment>
+</net>
