File: CAD/EEGAmp_SMT.brd (EAGLE design)
At the start: 21.6 x 11.2 mm, 14 parts, among them U1 TL084QD

Commit message: added a filter cap on inputs
Parts:
- added C4: 2.2nF, rcl:C0402
Connections:
- net 1IN-: now also C4.2
- net 2IN-: now also C4.1
Routing:
- net 2IN-: track 15.2 -> 16.9 mm
- net 1IN-: track 4.76 -> 6.01 mm
Changed lines of the file:
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@@
 <attribute name="VALUE" x="13.716" y="28.956" size="1.27" layer="27" rot="R270"/>
+</element>
+<element name="C4" library="rcl" library_urn="urn:adsk.eagle:library:334" package="C0402" package3d_urn="urn:adsk.eagle:package:23626/2" value="2.2nF" x="20.32" y="21.59" smashed="yes" rot="R270">
+<attribute name="NAME" x="20.828" y="22.733" size="1.27" layer="26" rot="MR270"/>
+<attribute name="POPULARITY" value="16" x="20.32" y="21.59" size="1.778" layer="27" rot="R270" display="off"/>
+<attribute name="SPICEPREFIX" value="C" x="20.32" y="21.59" size="1.778" layer="27" rot="R270" display="off"/>
 </element>
 </elements>
@@
 <contactref element="R4" pad="1"/>
 <wire x1="29.21" y1="22.925" x2="29.21" y2="20.701" width="0.1524" layer="1"/>
-<wire x1="28.6076" y1="20.0986" x2="21.4304" y2="20.0986" width="0.1524" layer="1"/>
-<wire x1="20.328" y1="21.201" x2="20.328" y2="23.495" width="0.1524" layer="1"/>
 <wire x1="29.21" y1="20.701" x2="28.6076" y2="20.0986" width="0.1524" layer="1"/>
-<wire x1="21.4304" y1="20.0986" x2="20.328" y2="21.201" width="0.1524" layer="1"/>
 <wire x1="20.328" y1="24.638" x2="20.328" y2="23.495" width="0.1524" layer="1"/>
+<contactref element="C4" pad="1"/>
+<wire x1="20.328" y1="23.495" x2="20.328" y2="22.248" width="0.1524" layer="1"/>
+<wire x1="20.328" y1="22.248" x2="20.32" y2="22.24" width="0.1524" layer="1"/>
+<wire x1="19.9064" y1="20.0986" x2="19.558" y2="20.447" width="0.1524" layer="1"/>
+<wire x1="19.558" y1="20.447" x2="19.558" y2="21.732" width="0.1524" layer="1"/>
+<wire x1="20.066" y1="22.24" x2="19.558" y2="21.732" width="0.1524" layer="1"/>
+<wire x1="20.066" y1="22.24" x2="20.32" y2="22.24" width="0.1524" layer="1"/>
+<wire x1="28.6076" y1="20.0986" x2="19.9064" y2="20.0986" width="0.1524" layer="1"/>
 </signal>
 <signal name="3IN+">
@@
 <wire x1="21.463" y1="21.217" x2="21.598" y2="21.082" width="0.1524" layer="1"/>
 <wire x1="21.598" y1="21.082" x2="24.265" y2="21.082" width="0.1524" layer="1"/>
+<contactref element="C4" pad="2"/>
+<wire x1="20.32" y1="20.94" x2="20.597" y2="21.217" width="0.1524" layer="1"/>
+<wire x1="20.597" y1="21.217" x2="21.463" y2="21.217" width="0.1524" layer="1"/>
 </signal>
 <signal name="4IN-">
