File: CAD/EEGAmp_SMT.sch (EAGLE design)
At the start: 14 parts, among them U1 TL084QD

Commit message: corrected notes
Other:
- note added: "VRef can be VDD or a dedicated voltage reference for the ADC"
- note removed: "VRef can be a voltage divider circuit if on battery power"
Changed lines of the file:
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@@
 R7: 1kΩ
 R8: 1MΩ</text>
-<text x="218.44" y="86.36" size="1.778" layer="97">VRef can be a voltage divider
-circuit if on battery power</text>
+<text x="218.44" y="86.36" size="1.778" layer="97">VRef can be VDD or a dedicated voltage reference for the ADC</text>
 </plain>
 <instances>

Commit message: added a filter cap on inputs
Parts:
- added C4: 2.2nF, rcl:C-USC0402
Connections:
- net 1IN-: now also C4.2
- net 2IN-: now also C4.1
Changed lines of the file:
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@@
 <part name="JP2" library="pinhead" library_urn="urn:adsk.eagle:library:325" deviceset="PINHD-1X4" device="" package3d_urn="urn:adsk.eagle:package:22407/2"/>
 <part name="JP3" library="pinhead" library_urn="urn:adsk.eagle:library:325" deviceset="PINHD-1X3" device="" package3d_urn="urn:adsk.eagle:package:22458/2"/>
+<part name="C4" library="rcl" library_urn="urn:adsk.eagle:library:334" deviceset="C-US" device="C0402" package3d_urn="urn:adsk.eagle:package:23626/2" value="2.2nF"/>
 </parts>
 <sheets>
@@
 <attribute name="VALUE" x="148.59" y="20.32" size="1.778" layer="96" rot="R180"/>
 </instance>
+<instance part="C4" gate="G$1" x="83.82" y="83.82" smashed="yes" rot="R270">
+<attribute name="NAME" x="84.836" y="81.915" size="1.778" layer="95"/>
+<attribute name="VALUE" x="79.756" y="79.629" size="1.778" layer="96"/>
+</instance>
 </instances>
 <busses>
@@
 <junction x="96.52" y="93.98"/>
 <label x="99.06" y="91.44" size="1.778" layer="95"/>
+</segment>
+<segment>
+<pinref part="C4" gate="G$1" pin="1"/>
+<wire x1="86.36" y1="83.82" x2="88.9" y2="83.82" width="0.1524" layer="91"/>
+<label x="88.9" y="83.82" size="1.778" layer="95"/>
 </segment>
 </net>
@@
 <junction x="60.96" y="93.98"/>
 </segment>
-</net>
+<segment>
+<pinref part="C4" gate="G$1" pin="2"/>
+<wire x1="78.74" y1="83.82" x2="76.2" y2="83.82" width="0.1524" layer="91"/>
+<label x="73.66" y="83.82" size="1.778" layer="95"/>
+</segment>
+</net>
